Commit message: Add n_robots namespacing and spawn spacing for MA-RPV* system.

File: src/vehicle_simulator/urdf/camera.urdf.xacro (robot description, xacro)
@@ -1,4 +1,8 @@
+<?xml version="1.0"?>
 <robot xmlns:xacro="http://www.ros.org/wiki/xacro" name="example">
-  <link name="camera">
+  <xacro:arg name="name" default="camera"/>
+  <xacro:arg name="ros_namespace" default=""/>
+  <xacro:arg name="frame_name" default="camera"/>
+  <link name="$(arg name)">
     <collision>
       <origin xyz="0 0 0" rpy="0 0 0"/>
@@ -19,6 +23,6 @@
     </inertial>
   </link>
-  <gazebo reference="camera">
-    <sensor type="camera" name="camera">
+  <gazebo reference="$(arg name)">
+    <sensor type="camera" name="$(arg name)_sensor">
       <update_rate>15.0</update_rate>
       <camera name="head">
@@ -34,5 +38,8 @@
         </clip>
       </camera>
-      <plugin name="camera_controller" filename="libgazebo_ros_camera.so">
+      <plugin name="$(arg name)_controller" filename="libgazebo_ros_camera.so">
+        <ros>
+          <namespace>$(arg ros_namespace)</namespace>
+        </ros>
         <alwaysOn>true</alwaysOn>
         <updateRate>0.0</updateRate>
@@ -40,5 +47,5 @@
         <imageTopicName>image</imageTopicName>
         <cameraInfoTopicName>camera_info</cameraInfoTopicName>
-        <frameName>camera</frameName>
+        <frameName>$(arg frame_name)</frameName>
         <hackBaseline>0.0</hackBaseline>
         <distortionK1>0.0</distortionK1>

File: src/vehicle_simulator/urdf/lidar.urdf.xacro (robot description, xacro)
@@ -1,7 +1,11 @@
 <?xml version="1.0"?>
 <robot xmlns:xacro="http://www.ros.org/wiki/xacro" name="example">
-  <link name="lidar" />
+  <xacro:arg name="scan_topic" default="/velodyne_points"/>
+  <xacro:arg name="tf_prefix" default=""/>
+  <xacro:arg name="sensor_name" default="velodyne"/>
+  <xacro:arg name="parent_link" default="lidar"/>
+  <link name="$(arg parent_link)" />
   <xacro:include filename="$(find velodyne_description)/urdf/VLP-16.urdf.xacro"/>
-  <xacro:VLP-16 parent="lidar" name="velodyne" topic="/velodyne_points" hz="6.3" samples="350" min_range="0.1" max_range="40.0">
+  <xacro:VLP-16 parent="$(arg parent_link)" name="$(arg sensor_name)" topic="$(arg scan_topic)" tf_prefix="$(arg tf_prefix)" hz="6.3" samples="350" min_range="0.1" max_range="40.0">
     <origin xyz="0 0 0" rpy="0 0 0" />
   </xacro:VLP-16>

File: src/vehicle_simulator/urdf_mp3d/lidar.urdf.xacro (robot description, xacro)
@@ -1,7 +1,11 @@
 <?xml version="1.0"?>
 <robot xmlns:xacro="http://www.ros.org/wiki/xacro" name="example">
-  <link name="lidar" />
+  <xacro:arg name="scan_topic" default="/velodyne_points"/>
+  <xacro:arg name="tf_prefix" default=""/>
+  <xacro:arg name="sensor_name" default="velodyne"/>
+  <xacro:arg name="parent_link" default="lidar"/>
+  <link name="$(arg parent_link)" />
   <xacro:include filename="$(find velodyne_description)/urdf/VLP-max.urdf.xacro"/>
-  <xacro:VLP-16 parent="lidar" name="velodyne" topic="/velodyne_points" hz="6.3" lasers="64" samples="720" min_range="0.001" max_range="10" gpu="true" collision_range="0.15">
+  <xacro:VLP-16 parent="$(arg parent_link)" name="$(arg sensor_name)" topic="$(arg scan_topic)" tf_prefix="$(arg tf_prefix)" hz="6.3" lasers="64" samples="720" min_range="0.001" max_range="10" gpu="true" collision_range="0.15">
     <origin xyz="0 0 0" rpy="0 0 0" />
   </xacro:VLP-16>
